Commit message: Build v04 stronger servo chassis with sampled sensors and revised policy rewards

File: simulation/generated/sweetie_mini.urdf (robot description, URDF)
Before this commit: robot sweetie_mini, 17 links, 16 joints
Links:
- added link chest_tof_frame
- added link forehead_rgb_frame
- added link torso_imu_frame
- link ear_left_link: mass 0.015885 -> 0.014253756081505371
- link ear_right_link: mass 0.015885 -> 0.014253756081505371
- link fl_roll_link: mass 0.11516 -> 0.3357009347534873; geometry collision box size=0.0335 0.044 0.0585; visual mesh filename=../../cad/STL/links/fl_roll.stl scale=.001 .001 .001
- link fl_shin_link: mass 0.054254 -> 0.11101100569021344; geometry collision box size=.03 .03 .0042; collision box size=0.016 0.003 0.038
- link fl_thigh_link: mass 0.111202 -> 0.3413365036047443; geometry collision box size=0.0335 0.044 0.0585; collision box size=0.038 0.003 0.131
- link fr_roll_link: mass 0.11516 -> 0.3357009347534873; geometry collision box size=0.0335 0.044 0.0585; visual mesh filename=../../cad/STL/links/fr_roll.stl scale=.001 .001 .001
- link fr_shin_link: mass 0.054254 -> 0.11101100569021344; geometry collision box size=.03 .03 .0042; collision box size=0.016 0.003 0.038
- link fr_thigh_link: mass 0.111202 -> 0.3413365036047443; geometry collision box size=0.0335 0.044 0.0585; collision box size=0.038 0.003 0.131
- link head_link: mass 0.34015799999999996 -> 0.2284621826823041; geometry collision box size=0.058 0.06 0.04; collision box size=0.092 0.086 0.086
- link neck_yaw_link: mass 0.116128 -> 0.13583667761005708
- link rl_roll_link: mass 0.11516 -> 0.3357009347534873; geometry collision box size=0.0335 0.044 0.0585; visual mesh filename=../../cad/STL/links/rl_roll.stl scale=.001 .001 .001
- link rl_shin_link: mass 0.054254 -> 0.11101100569021344; geometry collision box size=.03 .03 .0042; collision box size=0.016 0.003 0.038
- link rl_thigh_link: mass 0.111202 -> 0.3413365036047443; geometry collision box size=0.0335 0.044 0.0585; collision box size=0.038 0.003 0.131
- link rr_roll_link: mass 0.11516 -> 0.27760564784074865; geometry collision box size=0.0335 0.044 0.0585; visual mesh filename=../../cad/STL/links/rr_roll.stl scale=.001 .001 .001
- link rr_shin_link: mass 0.054254 -> 0.11101100569021344; geometry collision box size=.03 .03 .0042; collision box size=0.016 0.003 0.038
- link rr_thigh_link: mass 0.111202 -> 0.3413365036047443; geometry collision box size=0.0335 0.044 0.0585; collision box size=0.038 0.003 0.131
- link torso_link: mass 1.10084 -> 1.5745065954815036; geometry collision box size=0.034 0.0465 0.0285; collision box size=0.034 0.0465 0.0285
Joints:
- added joint chest_tof_mount: type fixed, parent torso_link, child chest_tof_frame, origin xyz=0.135 0 -0.01 rpy=0 0.3490658504 0
- added joint forehead_rgb_mount: type fixed, parent head_link, child forehead_rgb_frame, origin xyz=0.078 0 0.067 rpy=0 0 0
- added joint torso_imu_mount: type fixed, parent torso_link, child torso_imu_frame, origin xyz=0.01 0 0.029 rpy=0 0 0
- joint ear_left: limit lower=-0.25 upper=0.25 effort=1.955190875 velocity=5.69415 -> lower=-0.25 upper=0.25 effort=0.24271500000000004 velocity=11.635
- joint ear_right: limit lower=-0.25 upper=0.25 effort=1.955190875 velocity=5.69415 -> lower=-0.25 upper=0.25 effort=0.24271500000000004 velocity=11.635
- joint fl_hip_pitch: limit lower=-1.5 upper=1.1 effort=1.955190875 velocity=5.69415 -> lower=-1.5 upper=1.1 effort=6.270126843750001 velocity=4.869468613064179; origin xyz=0 0.018 -0.042 rpy=0 0 0 -> xyz=0 0.024 -0.05 rpy=0 0 0
- joint fl_hip_roll: limit lower=-0.55 upper=0.55 effort=1.955190875 velocity=5.69415 -> lower=-0.4 upper=0.4 effort=3.3440676500000004 velocity=5.031784233499652; origin xyz=0.086 0.052 0 rpy=0 0 0 -> xyz=0.099 0.058 0 rpy=0 0 0
- joint fl_knee: limit lower=0.1 upper=2.1 effort=1.955190875 velocity=5.69415 -> lower=0.1 upper=2.1 effort=6.270126843750001 velocity=4.869468613064179; origin xyz=0 0 -0.075 rpy=0 0 0 -> xyz=0 0 -0.095 rpy=0 0 0
- joint fr_hip_pitch: limit lower=-1.5 upper=1.1 effort=1.955190875 velocity=5.69415 -> lower=-1.5 upper=1.1 effort=6.270126843750001 velocity=4.869468613064179; origin xyz=0 -0.018 -0.042 rpy=0 0 0 -> xyz=0 -0.024 -0.05 rpy=0 0 0
- joint fr_hip_roll: limit lower=-0.55 upper=0.55 effort=1.955190875 velocity=5.69415 -> lower=-0.4 upper=0.4 effort=3.3440676500000004 velocity=5.031784233499652; origin xyz=0.086 -0.052 0 rpy=0 0 0 -> xyz=0.099 -0.058 0 rpy=0 0 0
- joint fr_knee: limit lower=0.1 upper=2.1 effort=1.955190875 velocity=5.69415 -> lower=0.1 upper=2.1 effort=6.270126843750001 velocity=4.869468613064179; origin xyz=0 0 -0.075 rpy=0 0 0 -> xyz=0 0 -0.095 rpy=0 0 0
- joint head_pitch: limit lower=-0.35 upper=0.35 effort=1.955190875 velocity=5.69415 -> lower=-0.35 upper=0.35 effort=2.090031625 velocity=6.08685
- joint head_yaw: limit lower=-0.8 upper=0.8 effort=1.955190875 velocity=5.69415 -> lower=-0.8 upper=0.8 effort=2.090031625 velocity=6.08685; origin xyz=0.082 0 0.014 rpy=0 0 0 -> xyz=0.096 0 0.014 rpy=0 0 0
- joint rl_hip_pitch: limit lower=-1.5 upper=1.1 effort=1.955190875 velocity=5.69415 -> lower=-1.5 upper=1.1 effort=6.270126843750001 velocity=4.869468613064179; origin xyz=0 0.018 -0.042 rpy=0 0 0 -> xyz=0 0.024 -0.05 rpy=0 0 0
- joint rl_hip_roll: limit lower=-0.55 upper=0.55 effort=1.955190875 velocity=5.69415 -> lower=-0.4 upper=0.4 effort=3.3440676500000004 velocity=5.031784233499652; origin xyz=-0.086 0.052 0 rpy=0 0 0 -> xyz=-0.099 0.058 0 rpy=0 0 0
- joint rl_knee: limit lower=0.1 upper=2.1 effort=1.955190875 velocity=5.69415 -> lower=0.1 upper=2.1 effort=6.270126843750001 velocity=4.869468613064179; origin xyz=0 0 -0.075 rpy=0 0 0 -> xyz=0 0 -0.095 rpy=0 0 0
- joint rr_hip_pitch: limit lower=-1.5 upper=1.1 effort=1.955190875 velocity=5.69415 -> lower=-1.5 upper=1.1 effort=6.270126843750001 velocity=4.869468613064179; origin xyz=0 -0.018 -0.042 rpy=0 0 0 -> xyz=0 -0.024 -0.05 rpy=0 0 0
- joint rr_hip_roll: limit lower=-0.55 upper=0.55 effort=1.955190875 velocity=5.69415 -> lower=-0.4 upper=0.4 effort=3.3440676500000004 velocity=5.031784233499652; origin xyz=-0.086 -0.052 0 rpy=0 0 0 -> xyz=-0.099 -0.058 0 rpy=0 0 0
- joint rr_knee: limit lower=0.1 upper=2.1 effort=1.955190875 velocity=5.69415 -> lower=0.1 upper=2.1 effort=6.270126843750001 velocity=4.869468613064179; origin xyz=0 0 -0.075 rpy=0 0 0 -> xyz=0 0 -0.095 rpy=0 0 0

Commit message: Redesign v05 mechanics and validate matching MuJoCo learning model

File: simulation/generated/sweetie_mini.urdf (robot description, URDF)
Before this commit: robot sweetie_mini, 20 links, 19 joints
Links:
- link ear_left_link: mass 0.014253756081505371 -> 0.014175350073357743; geometry collision mesh filename=../../cad/collision/convex/ear_left__ear_output_adapter_1__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 scale=.001 .001 .001; collision mesh filename=../../cad/collision/convex/ear_left__ear_shell_1__0.stl scale=.001 .001 .001
- link ear_right_link: mass 0.014253756081505371 -> 0.014175365078113157; geometry collision mesh filename=../../cad/collision/convex/ear_right__ear_output_adapter_-1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 scale=.001 .001 .001; collision mesh filename=../../cad/collision/convex/ear_right__ear_shell_-1__0.stl scale=.001 .001 .001
- link fl_roll_link: mass 0.3357009347534873 -> 0.474059733811006; geometry collision mesh filename=../../cad/collision/convex/fl_roll__fl_hip_bearing_retainer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 scale=.001 .001 .001; collision mesh filename=../../cad/collision/convex/fl_roll__fl_hip_bearing_retainer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 scale=.001 .001 .001
- link fl_shin_link: mass 0.11101100569021344 -> 0.19139004832181278; geometry collision box size=.03 .03 .0042; collision mesh filename=../../cad/collision/convex/fl_shin__fl_TPU_actuator__0.stl scale=.001 .001 .001
- link fl_thigh_link: mass 0.3413365036047443 -> 0.5016475672239777; geometry collision mesh filename=../../cad/collision/convex/fl_thigh__fl_hip_M3_heads_-68.0_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 scale=.001 .001 .001; collision mesh filename=../../cad/collision/convex/fl_thigh__fl_hip_M3_heads_-68.0_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 scale=.001 .001 .001
- link fr_roll_link: mass 0.3357009347534873 -> 0.4740597338110091; geometry collision mesh filename=../../cad/collision/convex/fr_roll__fr_hip_bearing_retainer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 scale=.001 .001 .001; collision mesh filename=../../cad/collision/convex/fr_roll__fr_hip_bearing_retainer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 scale=.001 .001 .001
- link fr_shin_link: mass 0.11101100569021344 -> 0.19139004831777717; geometry collision box size=.03 .03 .0042; collision mesh filename=../../cad/collision/convex/fr_shin__fr_TPU_actuator__0.stl scale=.001 .001 .001
- link fr_thigh_link: mass 0.3413365036047443 -> 0.501647567223975; geometry collision mesh filename=../../cad/collision/convex/fr_thigh__fr_hip_M3_heads_-8.0__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 scale=.001 .001 .001; collision mesh filename=../../cad/collision/convex/fr_thigh__fr_hip_M3_heads_-8.0__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 scale=.001 .001 .001
- link head_link: mass 0.2284621826823041 -> 0.26072589018361814; geometry collision mesh filename=../../cad/collision/convex/head__camera_board__0.stl scale=.001 .001 .001; collision mesh filename=../../cad/collision/convex/head__camera_carrier__0.stl scale=.001 .001 .001
- link neck_yaw_link: mass 0.13583667761005708 -> 0.17546671484734536; geometry collision mesh filename=../../cad/collision/convex/neck_yaw__head_pitch_clamp_shims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 scale=.001 .001 .001; collision mesh filename=../../cad/collision/convex/neck_yaw__head_pitch_clamp_shims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 scale=.001 .001 .001
- link rl_roll_link: mass 0.3357009347534873 -> 0.47405973381100697; geometry collision mesh filename=../../cad/collision/convex/rl_roll__rl_hip_bearing_retainer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 scale=.001 .001 .001; collision mesh filename=../../cad/collision/convex/rl_roll__rl_hip_bearing_retainer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 scale=.001 .001 .001
- link rl_shin_link: mass 0.11101100569021344 -> 0.19139004831765596; geometry collision box size=.03 .03 .0042; collision mesh filename=../../cad/collision/convex/rl_shin__rl_TPU_actuator__0.stl scale=.001 .001 .001
- link rl_thigh_link: mass 0.3413365036047443 -> 0.501647567223665; geometry collision mesh filename=../../cad/collision/convex/rl_thigh__rl_hip_M3_heads_-68.0_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 scale=.001 .001 .001; collision mesh filename=../../cad/collision/convex/rl_thigh__rl_hip_M3_heads_-68.0_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 scale=.001 .001 .001
- link rr_roll_link: mass 0.27760564784074865 -> 0.47405973381100724; geometry collision mesh filename=../../cad/collision/convex/rr_roll__rr_hip_bearing_retainer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 scale=.001 .001 .001; collision mesh filename=../../cad/collision/convex/rr_roll__rr_hip_bearing_retainer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 scale=.001 .001 .001
- link rr_shin_link: mass 0.11101100569021344 -> 0.1913900483216966; geometry collision box size=.03 .03 .0042; collision mesh filename=../../cad/collision/convex/rr_shin__rr_TPU_actuator__0.stl scale=.001 .001 .001
- link rr_thigh_link: mass 0.3413365036047443 -> 0.501647567223977; geometry collision mesh filename=../../cad/collision/convex/rr_thigh__rr_hip_M3_heads_-68.0_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 scale=.001 .001 .001; collision mesh filename=../../cad/collision/convex/rr_thigh__rr_hip_M3_heads_-68.0_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 scale=.001 .001 .001
- link torso_link: mass 1.5745065954815036 -> 2.23178963651774; geometry collision mesh filename=../../cad/collision/convex/torso__adapter_envelope__0.stl scale=.001 .001 .001; collision mesh filename=../../cad/collision/convex/torso__battery_envelope__0.stl scale=.001 .001 .001
Joints:
- joint ear_left: origin xyz=0.045 0.022 0.06 rpy=0 0 0 -> xyz=0.045 0.012 0.102 rpy=0 0 0
- joint ear_right: origin xyz=0.045 -0.022 0.06 rpy=0 0 0 -> xyz=0.045 -0.012 0.102 rpy=0 0 0
- joint fl_hip_pitch: limit lower=-1.5 upper=1.1 effort=6.270126843750001 velocity=4.869468613064179 -> lower=-1.5 upper=0.1 effort=6.270126843750001 velocity=4.869468613064179; origin xyz=0 0.024 -0.05 rpy=0 0 0 -> xyz=0 0.03 -0.062 rpy=0 0 0
- joint fl_hip_roll: limit lower=-0.4 upper=0.4 effort=3.3440676500000004 velocity=5.031784233499652 -> lower=-0.15 upper=0.15 effort=6.270126843750001 velocity=4.869468613064179; origin xyz=0.099 0.058 0 rpy=0 0 0 -> xyz=0.099 0.07 0 rpy=0 0 0
- joint fl_knee: origin xyz=0 0 -0.095 rpy=0 0 0 -> xyz=0 0 -0.115 rpy=0 0 0
- joint forehead_rgb_mount: origin xyz=0.078 0 0.067 rpy=0 0 0 -> xyz=0.078 0 0.091 rpy=0 0 0
- joint fr_hip_pitch: limit lower=-1.5 upper=1.1 effort=6.270126843750001 velocity=4.869468613064179 -> lower=-1.5 upper=0.1 effort=6.270126843750001 velocity=4.869468613064179; origin xyz=0 -0.024 -0.05 rpy=0 0 0 -> xyz=0 -0.03 -0.062 rpy=0 0 0
- joint fr_hip_roll: limit lower=-0.4 upper=0.4 effort=3.3440676500000004 velocity=5.031784233499652 -> lower=-0.15 upper=0.15 effort=6.270126843750001 velocity=4.869468613064179; origin xyz=0.099 -0.058 0 rpy=0 0 0 -> xyz=0.099 -0.07 0 rpy=0 0 0
- joint fr_knee: origin xyz=0 0 -0.095 rpy=0 0 0 -> xyz=0 0 -0.115 rpy=0 0 0
- joint head_pitch: origin xyz=0 0 0.044 rpy=0 0 0 -> xyz=0 0 0.048 rpy=0 0 0
- joint head_yaw: origin xyz=0.096 0 0.014 rpy=0 0 0 -> xyz=0.096 0 0.03 rpy=0 0 0
- joint rl_hip_pitch: axis 0 1 0 -> 0 -1 0; limit lower=-1.5 upper=1.1 effort=6.270126843750001 velocity=4.869468613064179 -> lower=-1.5 upper=0.1 effort=6.270126843750001 velocity=4.869468613064179; origin xyz=0 0.024 -0.05 rpy=0 0 0 -> xyz=0 0.03 -0.062 rpy=0 0 0
- joint rl_hip_roll: limit lower=-0.4 upper=0.4 effort=3.3440676500000004 velocity=5.031784233499652 -> lower=-0.15 upper=0.15 effort=6.270126843750001 velocity=4.869468613064179; origin xyz=-0.099 0.058 0 rpy=0 0 0 -> xyz=-0.099 0.07 0 rpy=0 0 0
- joint rl_knee: axis 0 1 0 -> 0 -1 0; origin xyz=0 0 -0.095 rpy=0 0 0 -> xyz=0 0 -0.115 rpy=0 0 0
- joint rr_hip_pitch: axis 0 1 0 -> 0 -1 0; limit lower=-1.5 upper=1.1 effort=6.270126843750001 velocity=4.869468613064179 -> lower=-1.5 upper=0.1 effort=6.270126843750001 velocity=4.869468613064179; origin xyz=0 -0.024 -0.05 rpy=0 0 0 -> xyz=0 -0.03 -0.062 rpy=0 0 0
- joint rr_hip_roll: limit lower=-0.4 upper=0.4 effort=3.3440676500000004 velocity=5.031784233499652 -> lower=-0.15 upper=0.15 effort=6.270126843750001 velocity=4.869468613064179; origin xyz=-0.099 -0.058 0 rpy=0 0 0 -> xyz=-0.099 -0.07 0 rpy=0 0 0
- joint rr_knee: axis 0 1 0 -> 0 -1 0; origin xyz=0 0 -0.095 rpy=0 0 0 -> xyz=0 0 -0.115 rpy=0 0 0

Commit message: Expand mirrored hip abduction for recovery with audited actor transfer

File: simulation/generated/sweetie_mini.urdf (robot description, URDF)
Before this commit: robot sweetie_mini, 20 links, 19 joints
Joints:
- joint fl_hip_roll: limit lower=-0.15 upper=0.15 effort=6.270126843750001 velocity=4.869468613064179 -> lower=-0.10471975511965978 upper=0.7853981633974483 effort=6.270126843750001 velocity=4.869468613064179
- joint fr_hip_roll: limit lower=-0.15 upper=0.15 effort=6.270126843750001 velocity=4.869468613064179 -> lower=-0.7853981633974483 upper=0.10471975511965978 effort=6.270126843750001 velocity=4.869468613064179
- joint rl_hip_roll: limit lower=-0.15 upper=0.15 effort=6.270126843750001 velocity=4.869468613064179 -> lower=-0.10471975511965978 upper=0.7853981633974483 effort=6.270126843750001 velocity=4.869468613064179
- joint rr_hip_roll: limit lower=-0.15 upper=0.15 effort=6.270126843750001 velocity=4.869468613064179 -> lower=-0.7853981633974483 upper=0.10471975511965978 effort=6.270126843750001 velocity=4.869468613064179
